File: hardware/smart-plant.kicad_pcb (KiCad board)
At the start: 2 copper layers, 41 x 75.3 mm, 28 parts, among them J1 USB_B_Micro, J2 Soil humidity sensor, J3 Water level sensor, J4 Display, M1 water pump, Q1 IRF540N, SW1 Button, SW2 Button, U1 L7805

Commit message: Add RTC
Parts:
- removed the REF** at (172.7, 80.4)
- removed the REF** at (157.7, 68.4)
- removed the REF** at (140.7, 96.0)
- removed the REF** at (161.7, 130.4)
- added BT1: Battery, smartplant:QJ-BS-6-1, B.Cu at (139.2, 102.0)
- added R10: 4k7, Resistor_SMD:R_1210_3225Metric_Pad1.30x2.65mm_HandSolder, F.Cu at (131.8, 94.8)
- added R11: 4k7, Resistor_SMD:R_1210_3225Metric_Pad1.30x2.65mm_HandSolder, F.Cu at (139.2, 126.0)
- added R12: 4k7, Resistor_SMD:R_1210_3225Metric_Pad1.30x2.65mm_HandSolder, F.Cu at (144.8, 126.0)
- added R8: 4k7, Resistor_SMD:R_1210_3225Metric_Pad1.30x2.65mm_HandSolder, F.Cu at (131.8, 90.6)
- added R9: 4k7, Resistor_SMD:R_1210_3225Metric_Pad1.30x2.65mm_HandSolder, F.Cu at (132.9, 86.3)
- added REF**: MountingHole_2.7mm_M2.5, MountingHole:MountingHole_2.7mm_M2.5, F.Cu at (139.2, 75.5)
- added REF**: MountingHole_2.7mm_M2.5, MountingHole:MountingHole_2.7mm_M2.5, F.Cu at (160.1, 69.0)
- added REF**: MountingHole_2.7mm_M2.5, MountingHole:MountingHole_2.7mm_M2.5, F.Cu at (160.1, 135.6)
- added REF**: MountingHole_2.7mm_M2.5, MountingHole:MountingHole_2.7mm_M2.5, F.Cu at (172.3, 81.0)
- added TP1: TestPoint, TestPoint:TestPoint_Pad_D1.0mm, F.Cu at (137.3, 105.0)
- added U2: DS1307ZN+, Package_SO:SOIC-8_3.9x4.9mm_P1.27mm, F.Cu at (132.7, 102.5)
- added Y1: 32.768 kHz, Crystal:Crystal_DS26_D2.0mm_L6.0mm_Horizontal, F.Cu at (130.4, 107.0)
- moved R1 10.6 mm to (168.8, 136.5), turned to 270 degrees
- moved C2 10.5 mm to (165.3, 136.5), turned to 270 degrees
- moved R2 9.38 mm to (161.9, 129.1)
- moved D2 7.29 mm to (143.4, 100.8), turned to 180 degrees
- moved J1 4.41 mm to (173.1, 130.4)
- moved M1 1.00 mm to (146.3, 81.7)
- moved C3 0.85 mm to (145.2, 75.2)
- moved J3 0.40 mm to (146.3, 71.4)
Connections:
- A1 pad 1: Net-(A1-Pad1) -> (no net)
- A1 pad 12: Net-(A1-Pad12) -> (no net)
- A1 pad 13: Net-(A1-Pad13) -> (no net)
- A1 pad 14: Net-(A1-Pad14) -> (no net)
- A1 pad 15: Net-(A1-Pad15) -> (no net)
- A1 pad 16: Net-(A1-Pad16) -> (no net)
- A1 pad 17: Net-(A1-Pad17) -> (no net)
- A1 pad 18: Net-(A1-Pad18) -> (no net)
- A1 pad 2: Net-(A1-Pad2) -> (no net)
- A1 pad 22: Net-(A1-Pad22) -> (no net)
- A1 pad 25: Net-(A1-Pad25) -> (no net)
- A1 pad 26: Net-(A1-Pad26) -> (no net)
- A1 pad 28: Net-(A1-Pad28) -> (no net)
- A1 pad 3: Net-(A1-Pad3) -> (no net)
- A1 pad 30: Net-(A1-Pad30) -> (no net)
- A1 pad 5: Net-(A1-Pad5) -> (no net)
- A1 pad 7: Net-(A1-Pad7) -> (no net)
- A1 pad 9: Net-(A1-Pad9) -> (no net)
- J1 pad 2: Net-(J1-Pad2) -> (no net)
- J1 pad 3: Net-(J1-Pad3) -> (no net)
- J1 pad 4: Net-(J1-Pad4) -> (no net)
Routing:
- net /SDA: track 51.1 -> 126.9 mm, vias 1 -> 2
- net /SCL: track 59.6 -> 118.0 mm, vias 1 -> 2
- net +5V: track 141.3 -> 196.7 mm
- net Net-(R10-Pad2): track 0.00 -> 14.9 mm
- net Net-(BT1-Pad1): track 0.00 -> 14.7 mm, vias 0 -> 1
- net Net-(C2-Pad1): track 35.2 -> 26.2 mm
- net /THERMISTOR: track 53.4 -> 60.5 mm
- net VBUS: track 85.2 -> 78.2 mm
- net GND: track 41.3 -> 44.9 mm, vias 18 -> 27
- net Net-(U2-Pad2): track 0.00 -> 2.21 mm
- net Net-(U2-Pad1): track 0.00 -> 2.20 mm
- net Net-(C4-Pad2): track 47.9 -> 47.1 mm, vias 1 -> 0
- added copper zone on F.Cu, net GND
Other:
- board size 41 x 75.3 mm -> 48 x 75.3 mm
