File: hardware/smart-plant.sch (KiCad schematic (older format))
At the start: 24 parts, among them J1 USB_B_Micro, J2 Soil humidity sensor, J3 Water level sensor, J4 Display, M1 water pump, Q1 IRF540N, SW1 Button, SW2 Button, U1 L7805

Commit message: Add RTC
Parts:
- added BT1: Battery, smartplant:QJ-BS-6-1, symbol Device:Battery_Cell
- added R10, R11, R12, R8, R9: 4k7, Resistor_SMD:R_1210_3225Metric_Pad1.30x2.65mm_HandSolder, symbol Device:R
- added TP1: TestPoint, TestPoint:TestPoint_Pad_D1.0mm, symbol Connector:TestPoint
- added U2: DS1307ZN+, Package_SO:SOIC-8_3.9x4.9mm_P1.27mm, symbol Timer_RTC:DS1307ZN+
- added Y1: 32.768 kHz, Crystal:Crystal_DS26_D2.0mm_L6.0mm_Horizontal, symbol Device:Crystal_Small
Connections:
- net +5V: now also R10.1, R11.1, R12.1, R8.1, R9.1, U2.8 (VCC)
- net GND: now also BT1.2 (-), U2.4 (GND)
- net SCL: now also R11.2, R8.2, U2.6 (SCL)
- net SDA: now also R12.2, R9.2, U2.5 (SDA)
- new net: U2.1 (X1), Y1.1
- new net: U2.2 (X2), Y1.2
- new net: BT1.1 (+), U2.3 (VBAT)
- new net: R10.2, TP1.1, U2.7 (SQW/OUT)
Other:
- moved on the sheet: J4
